Commit message: Update robot2.urdf

File: URDF/AR4_MK3/robot2.urdf (robot description, URDF)
Before this commit: robot robot_arm_urdf, 3 links, 2 joints
Links:
- added link gripper_jaw1_link, mass 0.5; collision mesh filename=C:/Users/MSI/python code/AR4_MK3/gripper_jaw1_link.STL; visual mesh filename=C:/Users/MSI/python code/AR4_MK3/gripper_jaw1_link.STL
- added link gripper_jaw2_link, mass 0.5; collision mesh filename=C:/Users/MSI/python code/AR4_MK3/gripper_jaw2_link.STL; visual mesh filename=C:/Users/MSI/python code/AR4_MK3/gripper_jaw2_link.STL
- added link gripper_link, mass 0.5; collision mesh filename=C:/Users/MSI/python code/AR4_MK3/gripper_base_link.STL; visual mesh filename=C:/Users/MSI/python code/AR4_MK3/gripper_base_link.STL
- added link link_3, mass 1.2; collision mesh filename=C:/Users/MSI/python code/AR4_MK3/link_3.STL; visual mesh filename=C:/Users/MSI/python code/AR4_MK3/link_3.STL
- added link link_4, mass 1.2; collision mesh filename=C:/Users/MSI/python code/AR4_MK3/link_4.STL; visual mesh filename=C:/Users/MSI/python code/AR4_MK3/link_4.STL
- added link link_5, mass 1.2; collision mesh filename=C:/Users/MSI/python code/AR4_MK3/link_5.STL; visual mesh filename=C:/Users/MSI/python code/AR4_MK3/link_5.STL
- added link link_6, mass 1.2; collision mesh filename=C:/Users/MSI/python code/AR4_MK3/link_6.STL; visual mesh filename=C:/Users/MSI/python code/AR4_MK3/link_6.STL
Joints:
- added joint gripper_jaw1_joint: type fixed, parent gripper_link, child gripper_jaw1_link, origin xyz=-0.020 -0.04 0 rpy=3.14 3.14 -3.14
- added joint gripper_jaw2_joint: type fixed, parent gripper_link, child gripper_jaw2_link, origin xyz=0.020 -0.039 0 rpy=3.14 0 3.14
- added joint gripper_joint: type fixed, parent link_6, child gripper_link, origin xyz=0 0 0 rpy=-1.57 0 0
- added joint joint_3: type continuous, parent link_2, child link_3, origin xyz=-0.0125 -.30 0 rpy=0 0 -3.14, axis 1 0 0, limit lower=-1.57 upper=1.57 effort=40 velocity=1.0
- added joint joint_4: type continuous, parent link_3, child link_4, origin xyz=0 0 0 rpy=0 -1.57 0, axis 1 0 0, limit lower=-1.57 upper=1.57 effort=40 velocity=1.0
- added joint joint_5: type revolute, parent link_4, child link_5, origin xyz=0 0 -.222 rpy=0 3.14 1.57, axis 1 0 0, limit lower=-1.57 upper=1.57 effort=40 velocity=1.0
- added joint joint_6: type revolute, parent link_5, child link_6, origin xyz=0 0 0.04 rpy=0 0 0, axis 1 0 0, limit lower=-1.57 upper=1.57 effort=40 velocity=1.0
- joint joint_2: origin xyz=0 0 0.5 rpy=0 0 0 -> xyz=0 0.07 -0.17 rpy=1.57 0 -1.57
